File: Kicad/Neotron-Expansion-Template.sch (KiCad schematic (older format))
At the start: 26 parts, among them J1 Neotron-Expansion-Edge, SW1 SW_DIP_x08, U1 MCP23S17, U2 34LC02

Commit message: Add kicad-exports.
Parts:
- C1, C2, C3, D1, D2, D3, D4, D5, D6, D7, D8, R1, R2, R3, R4, R5, R6, R7, R8, R9, SW1, U1, U2: DNP (none) -> 0
- J1, JP1: DNP (none) -> 1
- RN1: value 10k x 8 -> 10k; DNP (none) -> 0
Changed lines of the file:
@@
 F 2 "Neotron-Common-Hardware:Neotron-Expansion-Edge" H 6575 5800 50  0001 C CNN
 F 3 "" H 7025 5500 50  0001 C CNN
+F 4 "1" H 6575 5100 50  0001 C CNN "DNP"
 	1    6575 5100
 	1    0    0    -1
@@
 F 5 "Microchip" H 8200 5550 50  0001 C CNN "Manufacturer"
 F 6 "34LC02-I/P-ND" H 8200 5550 50  0001 C CNN "Digikey"
+F 7 "0" H 8200 5550 50  0001 C CNN "DNP"
 	1    8200 5550
 	1    0    0    -1
@@
 F 2 "Connector_PinHeader_2.54mm:PinHeader_1x02_P2.54mm_Vertical" H 9250 5875 50  0001 C CNN
 F 3 "~" H 9250 5875 50  0001 C CNN
+F 4 "1" H 9250 5875 50  0001 C CNN "DNP"
 	1    9250 5875
 	0    1    1    0
@@
 F 6 "C315C104M5U5TA" H 6000 6975 50  0001 C CNN "MPN"
 F 7 "KEMET" H 6000 6975 50  0001 C CNN "Manufacturer"
+F 8 "0" H 6000 6975 50  0001 C CNN "DNP"
 	1    6000 6975
 	1    0    0    -1
@@
 F 5 "Microchip" H 4525 4150 50  0001 C CNN "Manufacturer"
 F 6 "MCP23S17-E/SP-ND" H 4525 4150 50  0001 C CNN "Digikey"
+F 7 "0" H 4525 4150 50  0001 C CNN "DNP"
 	1    4525 4150
 	-1   0    0    1
@@
 F 5 "L314ED" H 2375 1300 50  0001 C CNN "MPN"
 F 6 "American Opto Plus LED" H 2375 1300 50  0001 C CNN "Manufacturer"
+F 7 "0" H 2375 1300 50  0001 C CNN "DNP"
 	1    2375 1300
 	1    0    0    -1
@@
 F 5 "CF14JT330R" H 2750 1300 50  0001 C CNN "MPN"
 F 6 "Stackpole Electronics Inc" H 2750 1300 50  0001 C CNN "Manufacturer"
+F 7 "0" H 2750 1300 50  0001 C CNN "DNP"
 	1    2750 1300
 	0    1    1    0
@@
 F 5 "CF14JT330R" H 2750 1600 50  0001 C CNN "MPN"
 F 6 "Stackpole Electronics Inc" H 2750 1600 50  0001 C CNN "Manufacturer"
+F 7 "0" H 2750 1600 50  0001 C CNN "DNP"
 	1    2750 1600
 	0    1    1    0
@@
 F 5 "CF14JT330R" H 2750 1900 50  0001 C CNN "MPN"
 F 6 "Stackpole Electronics Inc" H 2750 1900 50  0001 C CNN "Manufacturer"
+F 7 "0" H 2750 1900 50  0001 C CNN "DNP"
 	1    2750 1900
 	0    1    1    0
@@
 F 5 "CF14JT330R" H 2750 2200 50  0001 C CNN "MPN"
 F 6 "Stackpole Electronics Inc" H 2750 2200 50  0001 C CNN "Manufacturer"
+F 7 "0" H 2750 2200 50  0001 C CNN "DNP"
 	1    2750 2200
 	0    1    1    0
@@
 F 5 "CF14JT330R" H 2750 2500 50  0001 C CNN "MPN"
 F 6 "Stackpole Electronics Inc" H 2750 2500 50  0001 C CNN "Manufacturer"
+F 7 "0" H 2750 2500 50  0001 C CNN "DNP"
 	1    2750 2500
 	0    1    1    0
@@
 F 5 "CF14JT330R" H 2750 2800 50  0001 C CNN "MPN"
 F 6 "Stackpole Electronics Inc" H 2750 2800 50  0001 C CNN "Manufacturer"
+F 7 "0" H 2750 2800 50  0001 C CNN "DNP"
 	1    2750 2800
 	0    1    1    0
@@
 F 5 "CF14JT330R" H 2750 3100 50  0001 C CNN "MPN"
 F 6 "Stackpole Electronics Inc" H 2750 3100 50  0001 C CNN "Manufacturer"
+F 7 "0" H 2750 3100 50  0001 C CNN "DNP"
 	1    2750 3100
 	0    1    1    0
@@
 F 5 "CF14JT330R" H 2750 3400 50  0001 C CNN "MPN"
 F 6 "Stackpole Electronics Inc" H 2750 3400 50  0001 C CNN "Manufacturer"
+F 7 "0" H 2750 3400 50  0001 C CNN "DNP"
 	1    2750 3400
 	0    1    1    0
@@
 F 5 "L314ED" H 2375 1600 50  0001 C CNN "MPN"
 F 6 "American Opto Plus LED" H 2375 1600 50  0001 C CNN "Manufacturer"
+F 7 "0" H 2375 1600 50  0001 C CNN "DNP"
 	1    2375 1600
 	1    0    0    -1
@@
 F 5 "L314ED" H 2375 1900 50  0001 C CNN "MPN"
 F 6 "American Opto Plus LED" H 2375 1900 50  0001 C CNN "Manufacturer"
+F 7 "0" H 2375 1900 50  0001 C CNN "DNP"
 	1    2375 1900
 	1    0    0    -1
@@
 F 5 "L314ED" H 2375 2200 50  0001 C CNN "MPN"
 F 6 "American Opto Plus LED" H 2375 2200 50  0001 C CNN "Manufacturer"
+F 7 "0" H 2375 2200 50  0001 C CNN "DNP"
 	1    2375 2200
 	1    0    0    -1
@@
 F 5 "L314ED" H 2375 2500 50  0001 C CNN "MPN"
 F 6 "American Opto Plus LED" H 2375 2500 50  0001 C CNN "Manufacturer"
+F 7 "0" H 2375 2500 50  0001 C CNN "DNP"
 	1    2375 2500
 	1    0    0    -1
@@
 F 5 "L314ED" H 2375 2800 50  0001 C CNN "MPN"
 F 6 "American Opto Plus LED" H 2375 2800 50  0001 C CNN "Manufacturer"
+F 7 "0" H 2375 2800 50  0001 C CNN "DNP"
 	1    2375 2800
 	1    0    0    -1
@@
 F 5 "L314ED" H 2375 3100 50  0001 C CNN "MPN"
 F 6 "American Opto Plus LED" H 2375 3100 50  0001 C CNN "Manufacturer"
+F 7 "0" H 2375 3100 50  0001 C CNN "DNP"
 	1    2375 3100
 	1    0    0    -1
@@
 F 5 "L314ED" H 2375 3400 50  0001 C CNN "MPN"
 F 6 "American Opto Plus LED" H 2375 3400 50  0001 C CNN "Manufacturer"
+F 7 "0" H 2375 3400 50  0001 C CNN "DNP"
 	1    2375 3400
 	1    0    0    -1
@@
 F 6 "C315C104M5U5TA" H 6500 6975 50  0001 C CNN "MPN"
 F 7 "KEMET" H 6500 6975 50  0001 C CNN "Manufacturer"
+F 8 "0" H 6500 6975 50  0001 C CNN "DNP"
 	1    6500 6975
 	1    0    0    -1
@@
 F 6 "C315C104M5U5TA" H 5500 6975 50  0001 C CNN "MPN"
 F 7 "KEMET" H 5500 6975 50  0001 C CNN "Manufacturer"
+F 8 "0" H 5500 6975 50  0001 C CNN "DNP"
 	1    5500 6975
 	1    0    0    -1
@@
 F 5 "DS01C-254-L-08BE" H 2500 4650 50  0001 C CNN "MPN"
 F 6 "CUI Devices" H 2500 4650 50  0001 C CNN "Manufacturer"
+F 7 "0" H 2500 4650 50  0001 C CNN "DNP"
 	1    2500 4650
 	1    0    0    -1
@@
 F 5 "CF14JT10K0" H 9250 5400 50  0001 C CNN "MPN"
 F 6 "Stackpole Electronics Inc" H 9250 5400 50  0001 C CNN "Manufacturer"
+F 7 "0" H 9250 5400 50  0001 C CNN "DNP"
 	1    9250 5400
 	-1   0    0    1
@@
 P 3225 5325
 F 0 "RN1" H 3050 5600 50  0000 L CNN
-F 1 "10k x 8" H 3050 5525 50  0000 L CNN
+F 1 "10k" H 3050 5525 50  0000 L CNN
 F 2 "Resistor_THT:R_Array_SIP9" V 3700 5325 50  0001 C CNN
 F 3 "http://www.vishay.com/docs/31509/csc.pdf" H 3225 5325 50  0001 C CNN
@@
 F 5 "4609X-101-103LF" H 3225 5325 50  0001 C CNN "MPN"
 F 6 "4609X-101-103LF-ND" H 3225 5325 50  0001 C CNN "Digikey"
+F 7 "0" H 3225 5325 50  0001 C CNN "DNP"
 	1    3225 5325
 	-1   0    0    1
